File: cameraboard.kicad_sch (KiCad schematic)
At the start: 85 parts, among them J1 USB_C_Receptacle_USB2.0, J2 02x05 M 1.27mm, J3 Conn_01x08, J4 MOLEX_5051102491, J5 Conn_01x08, J6 TFM-110-12-X-D-A, J7 FLE-107-01-X-DV-A, J8 USD-1040310811, Q1 SQ3495EV-T1, SW1 CAS-120TA, SW2 KMR2x, SW3 CAS-120TA, U1 STM32H743VITx, U2 WE-TVS-82400102, U3 XC6210B332MR-G, U4 AP7366-28W5-7, U5 TLV75515PDBVR, U6 LTC4412xS6, Y1 16MHz

Commit message: Exported Gerbers
Parts:
- renumbered J8 to J3, J6 to J5, J7 to J6, J5 to J7, J3 to J8
Other:
- note added: "Select boot mode Set "low" for normal operation. Set "high" for bootloader mode"
- note added: "Set for flight"
Changed lines of the file:
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@@
     (effects (font (size 5.08 5.08)) (justify left bottom))
   )
+  (text "Set for flight" (at 254 157.607 0)
+    (effects (font (size 1.27 1.27)) (justify left bottom))
+  )
   (text "cameraboard" (at 335.534 263.525 0)
     (effects (font (size 3.81 3.81) (thickness 0.762) bold) (justify left bottom))
@@
     (effects (font (size 5.08 5.08)) (justify left bottom))
   )
+  (text "Set for flight" (at 170.053 177.038 0)
+    (effects (font (size 1.27 1.27)) (justify left bottom))
+  )
   (text "HI-Power\nSelection" (at 181.229 32.893 0)
     (effects (font (size 5.08 5.08)) (justify left bottom))
@@
     (effects (font (size 5.08 5.08)) (justify left bottom))
   )
+  (text "Select boot mode\nSet \"low\" for normal operation.\nSet \"high\" for bootloader mode"
+    (at 205.359 181.483 0)
+    (effects (font (size 1.27 1.27)) (justify left bottom))
+  )
   (text "USB Connector" (at 52.07 208.915 0)
     (effects (font (size 5.08 5.08)) (justify left bottom))
@@
   (symbol (lib_id "Connector_Generic:Conn_02x10_Odd_Even") (at 327.914 220.218 0) (unit 1)
     (in_bom yes) (on_board yes) (dnp no)
-    (property "Reference" "J6" (at 329.057 207.264 0)
+    (property "Reference" "J5" (at 329.057 207.264 0)
       (effects (font (size 1.27 1.27)))
     )
@@
       (project "cameraboard"
         (path "/71281620-6c96-40fb-9fa9-51f44fb772fb"
-          (reference "J6") (unit 1)
+          (reference "J5") (unit 1)
         )
       )
@@
   (symbol (lib_id "Connector_Generic:Conn_01x08") (at 290.068 232.918 0) (unit 1)
     (in_bom yes) (on_board no) (dnp yes)
-    (property "Reference" "J3" (at 288.925 219.964 0)
+    (property "Reference" "J8" (at 288.925 219.964 0)
       (effects (font (size 1.27 1.27)) (justify left))
     )
@@
       (project "cameraboard"
         (path "/71281620-6c96-40fb-9fa9-51f44fb772fb"
-          (reference "J3") (unit 1)
+          (reference "J8") (unit 1)
         )
       )
@@
   (symbol (lib_id "cameraboard:USD-1040310811") (at 378.333 150.114 0) (unit 1)
     (in_bom yes) (on_board yes) (dnp no)
-    (property "Reference" "J8" (at 370.713 129.286 0)
+    (property "Reference" "J3" (at 370.713 129.286 0)
       (effects (font (size 1.4986 1.4986)) (justify left bottom))
     )
@@
       (project "cameraboard"
         (path "/71281620-6c96-40fb-9fa9-51f44fb772fb"
-          (reference "J8") (unit 1)
+          (reference "J3") (unit 1)
         )
       )
@@
   (symbol (lib_id "Connector_Generic:Conn_01x08") (at 289.941 204.216 0) (unit 1)
     (in_bom yes) (on_board no) (dnp yes)
-    (property "Reference" "J5" (at 288.798 191.135 0)
+    (property "Reference" "J7" (at 288.798 191.135 0)
       (effects (font (size 1.27 1.27)) (justify left))
     )
@@
       (project "cameraboard"
         (path "/71281620-6c96-40fb-9fa9-51f44fb772fb"
-          (reference "J5") (unit 1)
+          (reference "J7") (unit 1)
         )
       )
@@
   (symbol (lib_id "Connector_Generic:Conn_02x07_Odd_Even") (at 378.079 217.932 0) (unit 1)
     (in_bom yes) (on_board yes) (dnp no)
-    (property "Reference" "J7" (at 379.349 207.645 0)
+    (property "Reference" "J6" (at 379.349 207.645 0)
       (effects (font (size 1.27 1.27)))
     )
@@
       (project "cameraboard"
         (path "/71281620-6c96-40fb-9fa9-51f44fb772fb"
-          (reference "J7") (unit 1)
+          (reference "J6") (unit 1)
         )
       )

Commit message: Rev B3/02 updates
Parts:
- removed FB2: 600R, Inductor_SMD:L_0603_1608Metric, symbol Device:FerriteBead_Small
- removed R5, R8: 22R, Resistor_SMD:R_0603_1608Metric, symbol Device:R_Small
- added R20: 0R, Resistor_SMD:R_0603_1608Metric, symbol Device:R_Small
- C16, C17: value 10pF -> 4pF
- H1, H2, H3, H4: now left out of the parts list
- Y1: value 16MHz -> 12MHz/7pF
- renumbered FB3 to FB2, R4 to R1, R20 to R10, R21 to R11, R11 to R12, R12 to R13, R13 to R14, R14 to R15, R15 to R17, R17 to R18, R18 to R19, R6 to R2, R7 to R3, R1 to R4, R3 to R5, R2 to R6, R9 to R7, R10 to R8, R19 to R9
Connections:
- net DC+ is gone; now on net D+: J1.A6 (D+), J1.B6 (D+)
- net DC- is gone; now on net D-: J1.A7 (D-), J1.B7 (D-)
- net VBUS: now also R20.2
- net at J1.A4 (VBUS), J1.A9 (VBUS), J1.B4 (VBUS)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: now also R20.1
Other:
- note added: "Check Xtal Datasheet This value assumes 7pF crystal bulk capacitance"
- note added: "Potentially Replace with Ferrite Bead"
