File: cameraboard.kicad_sch (KiCad schematic)
At the start: 83 parts, among them J1 USB_C_Receptacle_USB2.0, J2 02x05 M 1.27mm, J3 USD-1040310811, J4 MOLEX_5051102491, J5 TFM-110-12-X-D-A, J6 FLE-107-01-X-DV-A, J7 Conn_01x08, J8 Conn_01x08, Q1 SQ3495EV-T1, SW1 CAS-120TA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

Commit message: Rewired UART lines to mainboard
Parts:
- removed R17, R18: 4.7K, Resistor_SMD:R_0603_1608Metric, symbol Device:R_Small
- R15, R16: value 4.7K -> 10K
Connections:
- net 2.8V: no longer J4.1 (Pin_1)
- net GND: no longer J4.2 (Pin_2)
- net I2C2_SCL: no longer U1.46 (PB10)
- net I2C2_SDA: no longer U1.47 (PB11)
- net UART2_RX: no longer J5.5 (Pin_5)
- net UART2_TX: no longer J5.7 (Pin_7)
- new net UART3_RX: J5.5 (Pin_5), U1.47 (PB11)
- new net UART3_TX: J5.7 (Pin_7), U1.46 (PB10)
- no-connect marks 37 -> 39
Changed lines of the file:
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@@
   (title_block
     (title "PyCubed Mini")
-    (date "2023-04-12")
-    (rev "B3/02")
+    (date "2023-06-12")
+    (rev "B3/03")
     (company "REx Lab Carnegie Mellon University")
     (comment 1 "Z. Manchester")
@@
   (junction (at 221.361 221.869) (diameter 0) (color 0 0 0 0)
   )
-  (junction (at 335.153 33.02) (diameter 0) (color 0 0 0 0)
-  )
-  (junction (at 369.57 55.88) (diameter 0) (color 0 0 0 0)
-  )
   (junction (at 143.51 120.396) (diameter 0) (color 0 0 0 0)
   )
@@
   (junction (at 73.787 237.617) (diameter 0) (color 0 0 0 0)
   )
-  (junction (at 138.43 122.936) (diameter 0) (color 0 0 0 0)
-  )
   (junction (at 98.552 46.736) (diameter 0) (color 0 0 0 0)
   )
@@
   (junction (at 220.599 55.118) (diameter 0) (color 0 0 0 0)
   )
-  (junction (at 143.51 125.476) (diameter 0) (color 0 0 0 0)
-  )
   (junction (at 369.57 88.9) (diameter 0) (color 0 0 0 0)
   )
@@
   (no_connect (at 241.3 221.869))
   (no_connect (at 241.3 224.409))
+  (no_connect (at 384.81 35.56))
+  (no_connect (at 384.81 33.02))
   (no_connect (at 75.692 105.156))
   (no_connect (at 121.412 102.616))
@@
     (stroke (width 0) (type default))
   )
-  (wire (pts (xy 335.153 33.02) (xy 384.81 33.02))
-    (stroke (width 0) (type default))
-  )
   (wire (pts (xy 138.43 117.856) (xy 148.336 117.856))
     (stroke (width 0) (type default))
@@
     (stroke (width 0) (type default))
   )
-  (wire (pts (xy 328.803 33.02) (xy 335.153 33.02))
+  (wire (pts (xy 329.057 66.04) (xy 335.153 66.04))
     (stroke (width 0) (type default))
   )
@@
     (stroke (width 0) (type default))
   )
-  (wire (pts (xy 384.81 35.56) (xy 369.57 35.56))
-    (stroke (width 0) (type default))
-  )
   (wire (pts (xy 133.096 67.056) (xy 121.412 67.056))
     (stroke (width 0) (type default))
@@
     (stroke (width 0) (type default))
   )
-  (wire (pts (xy 121.412 125.476) (xy 143.51 125.476))
+  (wire (pts (xy 121.412 125.476) (xy 148.336 125.476))
     (stroke (width 0) (type default))
   )
@@
     (stroke (width 0) (type default))
   )
-  (wire (pts (xy 138.43 126.619) (xy 138.43 122.936))
-    (stroke (width 0) (type default))
-  )
   (wire (pts (xy 361.569 217.932) (xy 372.999 217.932))
     (stroke (width 0) (type default))
@@
     (stroke (width 0) (type default))
   )
-  (wire (pts (xy 121.412 122.936) (xy 138.43 122.936))
-    (stroke (width 0) (type default))
-  )
   (wire (pts (xy 123.571 44.958) (xy 123.571 46.609))
     (stroke (width 0) (type default))
@@
     (stroke (width 0) (type solid))
   )
-  (wire (pts (xy 138.43 122.936) (xy 148.336 122.936))
+  (wire (pts (xy 121.412 122.936) (xy 148.336 122.936))
     (stroke (width 0) (type default))
   )
@@
     (stroke (width 0) (type default))
   )
-  (wire (pts (xy 143.51 133.223) (xy 143.51 131.699))
-    (stroke (width 0) (type default))
-  )
   (wire (pts (xy 344.043 88.9) (xy 344.043 83.82))
     (stroke (width 0) (type default))
@@
     (stroke (width 0) (type default))
   )
-  (wire (pts (xy 335.153 33.02) (xy 335.153 66.04))
-    (stroke (width 0) (type default))
-  )
   (wire (pts (xy 296.037 77.978) (xy 296.037 79.375))
     (stroke (width 0) (type default))
@@
     (stroke (width 0) (type default))
   )
-  (wire (pts (xy 143.51 125.476) (xy 148.336 125.476))
-    (stroke (width 0) (type default))
-  )
   (wire (pts (xy 165.608 221.234) (xy 177.292 221.234))
     (stroke (width 0) (type default))
   )
-  (wire (pts (xy 369.57 35.56) (xy 369.57 55.88))
-    (stroke (width 0) (type default))
-  )
   (wire (pts (xy 211.963 70.739) (xy 207.899 70.739))
     (stroke (width 0) (type default))
@@
     (stroke (width 0) (type default))
   )
-  (wire (pts (xy 143.51 126.619) (xy 143.51 125.476))
-    (stroke (width 0) (type default))
-  )
   (wire (pts (xy 58.166 158.496) (xy 58.166 155.956))
     (stroke (width 0) (type solid))
@@
     (stroke (width 0) (type default))
   )
-  (wire (pts (xy 138.43 133.223) (xy 138.43 131.699))
-    (stroke (width 0) (type default))
-  )
   (wire (pts (xy 388.62 95.25) (xy 391.16 95.25))
     (stroke (width 0) (type default))
@@
     (effects (font (size 1.27 1.27)) (justify right bottom))
   )
-  (label "UART2_RX" (at 48.133 153.035 180) (fields_autoplaced)
+  (label "UART3_RX" (at 48.133 153.035 180) (fields_autoplaced)
     (effects (font (size 1.27 1.27)) (justify right bottom))
   )
@@
     (effects (font (size 1.27 1.27)) (justify left bottom))
   )
-  (label "UART2_TX" (at 48.133 155.575 180) (fields_autoplaced)
+  (label "UART3_TX" (at 48.133 155.575 180) (fields_autoplaced)
     (effects (font (size 1.27 1.27)) (justify right bottom))
   )
@@
     (effects (font (size 1.27 1.27)) (justify right bottom))
   )
-  (label "I2C2_SDA" (at 148.336 125.476 180) (fields_autoplaced)
+  (label "UART3_RX" (at 148.336 125.476 180) (fields_autoplaced)
     (effects (font (size 1.27 1.27)) (justify right bottom))
   )
@@
     (effects (font (size 1.27 1.27)) (justify left bottom))
   )
-  (label "I2C2_SCL" (at 148.336 122.936 180) (fields_autoplaced)
+  (label "UART3_TX" (at 148.336 122.936 180) (fields_autoplaced)
     (effects (font (size 1.27 1.27)) (justify right bottom))
   )
@@
     )
   )
-  (global_label "2.8V" (shape input) (at 328.803 33.02 180) (fields_autoplaced)
+  (global_label "2.8V" (shape input) (at 329.057 66.04 180) (fields_autoplaced)
     (effects (font (size 1.27 1.27)) (justify right))
-    (property "Intersheetrefs" "${INTERSHEET_REFS}" (at 322.2775 33.0994 0)
+    (property "Intersheetrefs" "${INTERSHEET_REFS}" (at 322.5315 66.1194 0)
       (effects (font (size 1.27 1.27)) (justify right) hide)
     )
@@
     )
   )
-  (symbol (lib_id "Device:R_Small") (at 143.51 129.159 180) (unit 1)
-    (in_bom yes) (on_board yes) (dnp no)
-    (property "Reference" "R18" (at 148.336 129.159 0)
-      (effects (font (size 1.27 1.27)) (justify left))
-    )
-    (property "Value" "4.7K" (at 143.51 127.762 90)
-      (effects (font (size 0.762 0.762)) (justify left))
-    )
-    (property "Footprint" "Resistor_SMD:R_0603_1608Metric" (at 143.51 129.159 0)
-      (effects (font (size 1.27 1.27)) hide)
-    )
-    (property "Datasheet" "~" (at 143.51 129.159 0)
-      (effects (font (size 1.27 1.27)) hide)
-    )
-    (pin "1")
-    (pin "2")
-    (instances
-      (project "cameraboard"
-        (path "/71281620-6c96-40fb-9fa9-51f44fb772fb"
-          (reference "R18") (unit 1)
-        )
-      )
-    )
-  )
   (symbol (lib_id "Device:C_Small") (at 252.222 104.394 0) (unit 1)
     (in_bom yes) (on_board yes) (dnp no)
@@
     )
   )
-  (symbol (lib_id "power:+3.3V") (at 138.43 133.223 180) (unit 1)
-    (in_bom yes) (on_board yes) (dnp no)
-    (property "Reference" "#PWR0155" (at 138.43 129.413 0)
-      (effects (font (size 1.27 1.27)) hide)
-    )
-    (property "Value" "+3.3V" (at 138.049 136.779 0)
-      (effects (font (size 1.27 1.27)))
-    )
-    (property "Footprint" "" (at 138.43 133.223 0)
-      (effects (font (size 1.27 1.27)) hide)
-    )
-    (property "Datasheet" "" (at 138.43 133.223 0)
-      (effects (font (size 1.27 1.27)) hide)
-    )
-    (pin "1")
-    (instances
-      (project "cameraboard"
-        (path "/71281620-6c96-40fb-9fa9-51f44fb772fb"
-          (reference "#PWR0155") (unit 1)
-        )
-      )
-    )
-  )
   (symbol (lib_id "Device:R_Small") (at 143.51 113.157 0) (unit 1)
     (in_bom yes) (on_board yes) (dnp no)
@@
       (effects (font (size 1.27 1.27)) (justify left))
     )
-    (property "Value" "4.7K" (at 143.51 114.554 90)
+    (property "Value" "10K" (at 143.51 114.3 90)
       (effects (font (size 0.762 0.762)) (justify left))
     )
@@
       (effects (font (size 1.27 1.27)) (justify left))
     )
-    (property "Value" "4.7K" (at 138.43 114.554 90)
+    (property "Value" "10K" (at 138.43 114.3 90)
       (effects (font (size 0.762 0.762)) (justify left))
     )
@@
       (effects (font (size 1.27 1.27)))
     )
-    (property "Value" "12MHz/7pF" (at 48.133 93.726 90)
+    (property "Value" "12MHz/7pF" (at 47.244 92.964 90)
       (effects (font (size 1.27 1.27)))
     )
@@
     )
   )
-  (symbol (lib_id "power:+3.3V") (at 143.51 133.223 180) (unit 1)
-    (in_bom yes) (on_board yes) (dnp no)
-    (property "Reference" "#PWR0157" (at 143.51 129.413 0)
-      (effects (font (size 1.27 1.27)) hide)
-    )
-    (property "Value" "+3.3V" (at 143.891 136.779 0)
-      (effects (font (size 1.27 1.27)))
-    )
-    (property "Footprint" "" (at 143.51 133.223 0)
-      (effects (font (size 1.27 1.27)) hide)
-    )
-    (property "Datasheet" "" (at 143.51 133.223 0)
-      (effects (font (size 1.27 1.27)) hide)
-    )
-    (pin "1")
-    (instances
-      (project "cameraboard"
-        (path "/71281620-6c96-40fb-9fa9-51f44fb772fb"
-          (reference "#PWR0157") (unit 1)
-        )
-      )
-    )
-  )
   (symbol (lib_id "power:GND") (at 335.153 95.25 0) (unit 1)
     (in_bom yes) (on_board yes) (dnp no)
@@
         )
       )
-    )
-  )
-  (symbol (lib_id "Device:R_Small") (at 138.43 129.159 180) (unit 1)
-    (in_bom yes) (on_board yes) (dnp no)
-    (property "Reference" "R17" (at 137.541 129.159 0)
-      (effects (font (size 1.27 1.27)) (justify left))
-    )
-    (property "Value" "4.7K" (at 138.43 127.762 90)
-      (effects (font (size 0.762 0.762)) (justify left))
-    )
-    (property "Footprint" "Resistor_SMD:R_0603_1608Metric" (at 138.43 129.159 0)
-      (effects (font (size 1.27 1.27)) hide)
-    )
-    (property "Datasheet" "~" (at 138.43 129.159 0)
-      (effects (font (size 1.27 1.27)) hide)
-    )
-    (pin "1")
-    (pin "2")
-    (instances
-      (project "cameraboard"
-        (path "/71281620-6c96-40fb-9fa9-51f44fb772fb"
-          (reference "R17") (unit 1)
-        )
-      )
